File: Winglet-EG800.kicad_sch (KiCad schematic)
At the start: 4 parts

Commit message: Update for DTR/DCD
Add LDO for 1v8 reference
Other:
- sheet Connector ports: added MODEM_DCD, MODEM_DTR; removed MODEM_PSM_IND, MODEM_PSM_INT
- sheet Modem ports: added MODEM_DCD, MODEM_DTR; removed MODEM_PSM_IND, MODEM_PSM_INT
Changed lines of the file:
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@@
 (kicad_sch
-	(version 20250114)
+	(version 20260306)
 	(generator "eeschema")
-	(generator_version "9.0")
+	(generator_version "10.0")
 	(paper "A4")
 	(title_block
 		(title "Winglet EG800")
-		(date "2026-03-03")
-		(rev "v1.0")
+		(date "2026-07-03")
+		(rev "v1.2")
 		(company "TL Embedded")
 	)
@@
 		(at 50.8 124.46 0)
 		(unit 1)
+		(body_style 1)
 		(exclude_from_sim no)
 		(in_bom no)
 		(on_board yes)
+		(in_pos_files yes)
 		(dnp no)
 		(fields_autoplaced yes)
 		(property "Reference" "N4"
 			(at 53.34 123.1899 0)
+			(show_name no)
+			(do_not_autoplace no)
 			(effects
 				(font
@@
 		(property "Value" "ToolingHole"
 			(at 53.34 125.7299 0)
+			(show_name no)
+			(do_not_autoplace no)
 			(effects
 				(font
@@
 		(property "Footprint" "N_NonPart:ToolingHole_1mm"
 			(at 51.054 129.54 0)
-			(effects
-				(font
-					(size 1.27 1.27)
-				)
-				(hide yes)
+			(hide yes)
+			(show_name no)
+			(do_not_autoplace no)
+			(effects
+				(font
+					(size 1.27 1.27)
+				)
 			)
 		)
 		(property "Datasheet" ""
 			(at 50.8 124.46 0)
-			(effects
-				(font
-					(size 1.27 1.27)
-				)
-				(hide yes)
+			(hide yes)
+			(show_name no)
+			(do_not_autoplace no)
+			(effects
+				(font
+					(size 1.27 1.27)
+				)
 			)
 		)
 		(property "Description" "TOOLING HOLE 1MM"
 			(at 50.8 131.318 0)
-			(effects
-				(font
-					(size 1.27 1.27)
-				)
-				(hide yes)
+			(hide yes)
+			(show_name no)
+			(do_not_autoplace no)
+			(effects
+				(font
+					(size 1.27 1.27)
+				)
 			)
 		)
@@
 		(at 49.53 138.43 0)
 		(unit 1)
+		(body_style 1)
 		(exclude_from_sim no)
 		(in_bom no)
 		(on_board yes)
+		(in_pos_files yes)
 		(dnp no)
 		(fields_autoplaced yes)
 		(property "Reference" "N1"
 			(at 59.69 132.7149 0)
+			(show_name no)
+			(do_not_autoplace no)
 			(effects
 				(font
@@
 		(property "Value" "QR 5mm"
 			(at 59.69 135.2549 0)
+			(show_name no)
+			(do_not_autoplace no)
 			(effects
 				(font
@@
 		(property "Footprint" "N_NonPart:QR_5mm_JLC"
 			(at 54.356 145.796 0)
-			(effects
-				(font
-					(size 1.27 1.27)
-				)
-				(hide yes)
+			(hide yes)
+			(show_name no)
+			(do_not_autoplace no)
+			(effects
+				(font
+					(size 1.27 1.27)
+				)
 			)
 		)
 		(property "Datasheet" ""
 			(at 48.895 139.065 0)
-			(effects
-				(font
-					(size 1.27 1.27)
-				)
-				(hide yes)
+			(hide yes)
+			(show_name no)
+			(do_not_autoplace no)
+			(effects
+				(font
+					(size 1.27 1.27)
+				)
 			)
 		)
 		(property "Description" "QR 8mm JLCPCB"
 			(at 54.102 143.764 0)
-			(effects
-				(font
-					(size 1.27 1.27)
-				)
-				(hide yes)
+			(hide yes)
+			(show_name no)
+			(do_not_autoplace no)
+			(effects
+				(font
+					(size 1.27 1.27)
+				)
 			)
 		)
 		(instances
-			(project ""
+			(project "Winglet-EG800"
 				(path "/332623d6-c22a-48da-966b-0d541566aa2d"
 					(reference "N1")
@@
 		(at 50.8 119.38 0)
 		(unit 1)
+		(body_style 1)
 		(exclude_from_sim no)
 		(in_bom no)
 		(on_board yes)
+		(in_pos_files yes)
 		(dnp no)
 		(fields_autoplaced yes)
 		(property "Reference" "N3"
 			(at 53.34 118.1099 0)
+			(show_name no)
+			(do_not_autoplace no)
 			(effects
 				(font
@@
 		(property "Value" "ToolingHole"
 			(at 53.34 120.6499 0)
+			(show_name no)
+			(do_not_autoplace no)
 			(effects
 				(font
@@
 		(property "Footprint" "N_NonPart:ToolingHole_1mm"
 			(at 51.054 124.46 0)
-			(effects
-				(font
-					(size 1.27 1.27)
-				)
-				(hide yes)
+			(hide yes)
+			(show_name no)
+			(do_not_autoplace no)
+			(effects
+				(font
+					(size 1.27 1.27)
+				)
 			)
 		)
 		(property "Datasheet" ""
 			(at 50.8 119.38 0)
-			(effects
-				(font
-					(size 1.27 1.27)
-				)
-				(hide yes)
+			(hide yes)
+			(show_name no)
+			(do_not_autoplace no)
+			(effects
+				(font
+					(size 1.27 1.27)
+				)
 			)
 		)
 		(property "Description" "TOOLING HOLE 1MM"
 			(at 50.8 126.238 0)
-			(effects
-				(font
-					(size 1.27 1.27)
-				)
-				(hide yes)
+			(hide yes)
+			(show_name no)
+			(do_not_autoplace no)
+			(effects
+				(font
+					(size 1.27 1.27)
+				)
 			)
 		)
@@
 		(at 50.8 114.3 0)
 		(unit 1)
+		(body_style 1)
 		(exclude_from_sim no)
 		(in_bom no)
 		(on_board yes)
+		(in_pos_files yes)
 		(dnp no)
 		(fields_autoplaced yes)
 		(property "Reference" "N2"
 			(at 53.34 113.0299 0)
+			(show_name no)
+			(do_not_autoplace no)
 			(effects
 				(font
@@
 		(property "Value" "ToolingHole"
 			(at 53.34 115.5699 0)
+			(show_name no)
+			(do_not_autoplace no)
 			(effects
 				(font
@@
 		(property "Footprint" "N_NonPart:ToolingHole_1mm"
 			(at 51.054 119.38 0)
-			(effects
-				(font
-					(size 1.27 1.27)
-				)
-				(hide yes)
+			(hide yes)
+			(show_name no)
+			(do_not_autoplace no)
+			(effects
+				(font
+					(size 1.27 1.27)
+				)
 			)
 		)
 		(property "Datasheet" ""
 			(at 50.8 114.3 0)
-			(effects
-				(font
-					(size 1.27 1.27)
-				)
-				(hide yes)
+			(hide yes)
+			(show_name no)
+			(do_not_autoplace no)
+			(effects
+				(font
+					(size 1.27 1.27)
+				)
 			)
 		)
 		(property "Description" "TOOLING HOLE 1MM"
 			(at 50.8 121.158 0)
-			(effects
-				(font
-					(size 1.27 1.27)
-				)
-				(hide yes)
+			(hide yes)
+			(show_name no)
+			(do_not_autoplace no)
+			(effects
+				(font
+					(size 1.27 1.27)
+				)
 			)
 		)
 		(instances
-			(project ""
+			(project "Winglet-EG800"
 				(path "/332623d6-c22a-48da-966b-0d541566aa2d"
 					(reference "N2")
@@
 		)
 		(fill
-			(color 175 255 191 1.0000)
+			(color 175 255 191 1)
 		)
 		(property "Sheetname" "Connector"
 			(at 38.1 37.3884 0)
+			(show_name no)
+			(do_not_autoplace no)
 			(effects
 				(font
@@
 		(property "Sheetfile" "connector.kicad_sch"
 			(at 38.1 102.1846 0)
+			(show_name no)
+			(do_not_autoplace no)
 			(effects
 				(font
@@
 			)
 		)
-		(pin "MODEM_PSM_IND" input
+		(pin "MODEM_DCD" input
 			(at 63.5 46.99 0)
 			(effects
@@
 			)
 		)
-		(pin "MODEM_PSM_INT" output
+		(pin "MODEM_DTR" output
 			(at 63.5 49.53 0)
 			(effects
@@
 		)
 		(fill
-			(color 175 255 191 1.0000)
+			(color 175 255 191 1)
 		)
 		(property "Sheetname" "Modem"
 			(at 152.4 37.3884 0)
+			(show_name no)
+			(do_not_autoplace no)
 			(effects
 				(font
@@
 		(property "Sheetfile" "modem.kicad_sch"
 			(at 152.4 102.1846 0)
+			(show_name no)
+			(do_not_autoplace no)
 			(effects
 				(font
@@
 			)
 		)
-		(pin "MODEM_PSM_IND" output
+		(pin "MODEM_DCD" output
 			(at 152.4 46.99 180)
 			(effects
@@
 			)
 		)
-		(pin "MODEM_PSM_INT" input
+		(pin "MODEM_DTR" input
 			(at 152.4 49.53 180)
 			(effects
@@
 		)
 		(fill
-			(color 175 255 191 1.0000)
+			(color 175 255 191 1)
 		)
 		(property "Sheetname" "Memory"
 			(at 88.9 85.6484 0)
+			(show_name no)
+			(do_not_autoplace no)
 			(effects
 				(font
@@
 		(property "Sheetfile" "memory.kicad_sch"
 			(at 88.9 102.1846 0)
-			(effects
-				(font
+			(show_name no)
+			(do_not_autoplace no)
+			(effects
+				(font
