File: memory.kicad_sch (KiCad schematic)
At the start: 10 parts, among them J2 NSIM-16-B, U3 MFF2-SIM, U4 24AA01T-I/OT

Commit message: Update for DTR/DCD
Add LDO for 1v8 reference
Parts:
- renumbered C8 to C10, C9 to C11, C10 to C12, C11 to C13, C12 to C14, C7 to C9, R3 to R4, U3 to U4, U4 to U5
