File: modem.kicad_sch (KiCad schematic)
At the start: 14 parts, among them J1 2337019-1, U2 EG800QEULC-N03-SNNSA

Commit message: Update for DTR/DCD
Add LDO for 1v8 reference
Parts:
- removed TP4: ~, TP_TestPoint:TestPoint_1mm, symbol TP_TestPoint:TestPoint_1mm
- added TP1, TP2, TP6: (no value), TP_TestPoint:TestPoint_1mm, symbol TP_TestPoint:TestPoint_1mm
- TP3: renamed from TP6; value ~ -> (none)
- TP4: renamed from TP7; value ~ -> (none)
- TP5: value ~ -> (none)
- TP7: renamed from TP1; value ~ -> (none)
- TP8: renamed from TP2; value ~ -> (none)
- TP9: renamed from TP3; value ~ -> (none)
- renumbered C3 to C5, C4 to C6, C5 to C7, C6 to C8, U2 to U3
Connections:
- net MODEM_DTR: now reaches U3.19 (MAIN_DTR)
- net MODEM_DTR: now also TP1.1
- net MODEM_DCD: now reaches U3.21 (MAIN_DCD)
- net MODEM_DCD: now also TP2.1
- net +1V8 renamed +1V8_MODEM
- net MODEM_PSM_IND: no longer names the net of U3.83 (PSM_IND)
- net MODEM_PSM_IND: now also TP5.1
- net MODEM_PSM_INT: no longer names the net of U3.87 (PSM_INT)
- net MODEM_PSM_INT: now also TP6.1; no longer TP5.1
- no-connect marks 17 -> 15
