File: Winglet-EG800.kicad_pcb (KiCad board)
At the start: 4 copper layers, 30 x 47.6 mm, 40 parts, among them J1 2337019-1, J2 NSIM-16-B, M1 PTH_M2.5, M2 PTH_M2.5, Q1 DMG1012UW-7, Q2 DMG1012UW-7, U1 FXLA108BQX, U2 EG800QEULC-N03-SNNSA, U3 MFF2-SIM, U4 24AA01T-I/OT

Commit message: Update for DTR/DCD
Add LDO for 1v8 reference
Parts:
- removed the TP4 at (57.5, 83.5)
- added C1: 100n, C_Capacitor:C_0603, F.Cu at (53.2, 81.0)
- added C2: 100n, C_Capacitor:C_0603, F.Cu at (53.2, 86.5)
- added R1: 0R, R_Resistor:R_0603, F.Cu at (53.2, 88.0)
- added TP1: ~, TP_TestPoint:TestPoint_1mm, F.Cu at (57.5, 86.0)
- added TP2: ~, TP_TestPoint:TestPoint_1mm, F.Cu at (57.5, 83.5)
- added TP6: ~, TP_TestPoint:TestPoint_1mm, F.Cu at (54.0, 66.6)
- added U1: MCP1711T-18I/OT, U_IC:SOT23_5, F.Cu at (53.2, 83.7)
- MP1: renamed from M1; footprint M_Mechanical:PTH_M2.5 -> MP_Mechanical:PTH_M2.5
- MP2: renamed from M2; footprint M_Mechanical:PTH_M2.5 -> MP_Mechanical:PTH_M2.5
- moved TP5 17.1 mm to (54.0, 69.3)
- moved TP8 2.99 mm to (54.0, 61.1)
- moved TP9 2.55 mm to (54.0, 58.4)
- moved R2 1.60 mm to (52.4, 75.0)
- moved R3 1.60 mm to (52.4, 78.0)
- moved Q1 1.60 mm to (54.8, 75.0)
- moved Q2 1.60 mm to (54.8, 78.0)
- moved TP7 0.28 mm to (54.0, 63.8)
- renumbered C8 to C10, C9 to C11, C10 to C12, C11 to C13, C12 to C14, C1 to C3, C2 to C4, C3 to C5, C4 to C6, C5 to C7, C6 to C8, C7 to C9, R1 to R2, R2 to R3, R3 to R4, TP6 to TP3, TP7 to TP4, TP1 to TP7, TP2 to TP8, TP3 to TP9, U1 to U2, U2 to U3, U3 to U4, U4 to U5
Connections:
- TP3 pad 1: +1V8 -> +1V8_MODEM
- TP5 pad 1: /Connector/MODEM_PSM_INT -> Net-(U3A-PSM_IND)
- U2 pad 13: /Connector/MODEM_PSM_IND -> /Connector/MODEM_DCD
- U2 pad 14: /Connector/MODEM_PSM_INT -> /Connector/MODEM_DTR
- U3 pad 19: unconnected-(U2A-MAIN_DTR-Pad19) -> /Connector/MODEM_DTR
- U3 pad 21: unconnected-(U2A-MAIN_DCD-Pad21) -> /Connector/MODEM_DCD
- U3 pad 24: +1V8 -> +1V8_MODEM
- U3 pad 83: /Connector/MODEM_PSM_IND -> Net-(U3A-PSM_IND)
- U3 pad 87: /Connector/MODEM_PSM_INT -> Net-(U3A-PSM_INT)
Routing:
- net +1V8_MODEM: track 0.00 -> 39.0 mm, vias 0 -> 2
- net /Connector/MODEM_PSM_INT: track 36.7 -> 0.00 mm, vias 2 -> 0
- net +1V8: track 40.7 -> 8.65 mm, vias 2 -> 0
- net /Connector/MODEM_PSM_IND: track 31.7 -> 0.00 mm, vias 2 -> 0
- net /Connector/MODEM_DCD: track 0.00 -> 26.0 mm, vias 0 -> 2
- net +BATT: track 2.94 -> 27.4 mm, vias 9 -> 11
- net /Connector/MODEM_DTR: track 0.00 -> 24.3 mm, vias 0 -> 2
- net Net-(U3A-PSM_INT): track 0.00 -> 21.8 mm, vias 0 -> 2
- net Net-(U3A-PSM_IND): track 0.00 -> 15.9 mm, vias 0 -> 2
- net /Connector/MODEM_AUX_TX: track 45.1 -> 37.8 mm
- net /Connector/MODEM_AUX_RX: track 47.9 -> 40.8 mm
- net /Connector/WAKE: track 23.3 -> 25.9 mm, vias 0 -> 2
- net /Connector/RESET: track 33.8 -> 35.8 mm
- net /Connector/MODEM_RESET: track 10.4 -> 8.41 mm
- net GND: track 39.8 -> 41.7 mm, vias 152 -> 126
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Other:
- board text added: "Winglet-EG800 v1.2 Jul 26"
- board text removed: "Winglet-EG800 v1.0 Mar 26"

Commit message: Add via stitching
Routing:
- net GND: vias 126 -> 157
